File: vfd_stm32/Logic.sch (KiCad schematic (older format))
At the start: 1 part

Commit message: routage terminé
Parts:
- added SW1: SW_DIP_x04, Button_Switch_SMD:SW_DIP_SPSTx04_Slide_6.7x11.72mm_W6.73mm_P2.54mm_LowProfile_JPin, symbol Switch:SW_DIP_x04
- gave numbers to parts that had none: 1
Connections:
- net labels added: Select_Master_Slave
- wire segments 3 -> 6
- no-connect marks 0 -> 3
Changed lines of the file:
@@
 $EndComp
 $Comp
-L MCU_ST_STM32F3:STM32F302C8Tx U?
+L MCU_ST_STM32F3:STM32F302C8Tx U20
 U 1 1 5DD8F475
 P 4500 3650
-F 0 "U?" H 5050 5000 50  0000 C CNN
+F 0 "U20" H 5050 5000 50  0000 C CNN
 F 1 "STM32F302C8Tx" H 4650 4550 50  0000 C CNN
 F 2 "Package_QFP:LQFP-48_7x7mm_P0.5mm" H 3900 2250 50  0001 R CNN
@@
 $EndComp
 $Comp
-L power:GND #PWR?
+L power:GND #PWR0136
 U 1 1 5DD9166A
 P 4500 5150
-F 0 "#PWR?" H 4500 4900 50  0001 C CNN
+F 0 "#PWR0136" H 4500 4900 50  0001 C CNN
 F 1 "GND" H 4505 4977 50  0000 C CNN
 F 2 "" H 4500 5150 50  0001 C CNN
@@
 Wire Wire Line
 	4500 5150 4600 5150
+Text Label 7350 1400 2    50   ~ 0
+Select_Master_Slave
+NoConn ~ 7350 1700
+NoConn ~ 7350 1600
+NoConn ~ 7350 1500
+$Comp
+L Switch:SW_DIP_x04 SW?
+U 1 1 5DDB47FF
+P 7650 1600
+AR Path="/5DDB47FF" Ref="SW?"  Part="1"
+AR Path="/5C025ADD/5DDB47FF" Ref="SW1"  Part="1"
+F 0 "SW1" H 7650 2067 50  0000 C CNN
+F 1 "SW_DIP_x04" H 7650 1976 50  0000 C CNN
+F 2 "Button_Switch_SMD:SW_DIP_SPSTx04_Slide_6.7x11.72mm_W6.73mm_P2.54mm_LowProfile_JPin" H 7650 1600 50  0001 C CNN
+F 3 "" H 7650 1600 50  0001 C CNN
+	1    7650 1600
+	1    0    0    -1
+$EndComp
+Wire Wire Line
+	7950 1400 7950 1500
+Connection ~ 7950 1500
+Wire Wire Line
+	7950 1500 7950 1600
+Connection ~ 7950 1600
+Wire Wire Line
+	7950 1600 7950 1700
+$Comp
+L power:GND #PWR?
+U 1 1 5DDB480B
+P 7950 1700
+AR Path="/5DDB480B" Ref="#PWR?"  Part="1"
+AR Path="/5C025ADD/5DDB480B" Ref="#PWR0142"  Part="1"
+F 0 "#PWR0142" H 7950 1450 50  0001 C CNN
+F 1 "GND" H 7950 1550 50  0000 C CNN
+F 2 "" H 7950 1700 50  0001 C CNN
+F 3 "" H 7950 1700 50  0001 C CNN
+	1    7950 1700
+	1    0    0    -1
+$EndComp
+Connection ~ 7950 1700
 $EndSCHEMATC
