File: vfd_stm32/Logic.sch (KiCad schematic (older format))
At the start: 2 parts, among them SW1 SW_DIP_x04, U20 STM32F302C8Tx

Commit message: continue circuitry
Connections:
- net labels added: Filament_Current_ADC, Filament_Enable, Filament_PWM1, Filament_PWM2, Grids_Anodes_SPI_MOSI, Grids_Anodes_SPI_RCLK, Grids_Anodes_SPI_SRCLK
Changed lines of the file:
@@
 $Descr A4 11693 8268
 encoding utf-8
-Sheet 3 3
+Sheet 3 4
 Title ""
 Date ""
@@
 $EndComp
 Connection ~ 7950 1700
+Text HLabel 7900 3500 2    50   Input ~ 0
+Filament_PWM2
+Text HLabel 7900 3600 2    50   Input ~ 0
+Filament_Enable
+Text HLabel 7900 3400 2    50   Input ~ 0
+Filament_PWM1
+Text HLabel 7900 3700 2    50   Input ~ 0
+Filament_Current_ADC
+Text HLabel 7900 4100 2    50   Input ~ 0
+Grids_Anodes_SPI_RCLK
+Text HLabel 7900 4000 2    50   Input ~ 0
+Grids_Anodes_SPI_MOSI
+Text HLabel 7900 4200 2    50   Input ~ 0
+Grids_Anodes_SPI_SRCLK
 $EndSCHEMATC
