File: vfd_stm32/VFD.sch (KiCad schematic (older format))
At the start: 10 parts

Commit message: cleanup electronics
Parts:
- added C10, C11, C4, C5, C6, C7, C8, C9: 100n, Capacitor_SMD:C_0805_2012Metric_Pad1.15x1.40mm_HandSolder, symbol Device:C
- added U10, U11, U12, U13, U2, U3, U4, U5: 74HC595, Package_SO:SOIC-16_3.9x9.9mm_P1.27mm, symbol 74xx:74HC595
- U14, U15, U16, U17, U6, U7, U8, U9: renamed from U?; footprint (none) -> Package_SO:SOIC-16_3.9x9.9mm_P1.27mm
- gave numbers to parts that had none: 1
Connections:
- net labels added: Power_Grids_Anodes, RCLK, SPI_Grids_Anodes_A, SPI_Grids_Anodes_B, SRCLK, VCC
- net labels removed: 35V
- wire segments 166 -> 248
- no-connect marks 5 -> 12
Other:
- moved on the sheet: U15, U16, U17, U1A, U6, U7, U8, U9

Commit message: routage terminé
Parts:
- removed U12, U13: 74HC595, Package_SO:SOIC-16_3.9x9.9mm_P1.27mm, symbol 74xx:74HC595
- added U16, U17: 74HC595, Package_SO:SOIC-16_3.9x9.9mm_P1.27mm, symbol 74xx:74HC595
- renumbered U2 to U10, U3 to U11, U4 to U12, U5 to U13, U10 to U14, U11 to U15, U7 to U2, U8 to U3, U9 to U4, U14 to U5, U15 to U6, U16 to U7, U17 to U8, U6 to U9
Connections:
- net labels added: G1, G10, G11, G12, G13, G14, G15, G16, G17, G18, G19, G2, G20, G3, G4, G5, G6, G7, G8, G9, P1, P10, P11, P12, P13, P14, P15, P16, P17, P18, P19, P2, P20, P21, P22, P23, P24, P25, P26, P27, P28, P29, P3, P30, P31, P32, P33, P34, P35, P4, P5, P6, P7, P8, P9
- net labels removed: SPI_Grids_Anodes_B
- wire segments 248 -> 193
Other:
- moved on the sheet: C4, C5, C6, C7, C8, C9, U1A, U1B, U2, U3, U4, U5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

Commit message: Fix shift registers outputs. Add text description files
Changed lines of the file:
@@
 Wire Wire Line
 	-2200 10550 -2200 10800
-Text Label -1400 5500 0    50   ~ 0
+Text Label -1400 5700 0    50   ~ 0
 G11
-Text Label -1400 5400 0    50   ~ 0
+Text Label -1400 5600 0    50   ~ 0
 G12
 Wire Wire Line
@@
 Wire Wire Line
 	-1350 4700 -1400 4700
+Text Label -1400 5500 0    50   ~ 0
+G13
+Text Label -1400 5400 0    50   ~ 0
+G14
 Text Label -1400 5300 0    50   ~ 0
-G13
+G15
 Text Label -1400 5200 0    50   ~ 0
-G14
+G16
 Text Label -1400 4500 0    50   ~ 0
-G15
-Text Label -1400 4400 0    50   ~ 0
-G16
-Text Label -1400 4300 0    50   ~ 0
 G17
 NoConn ~ -1400 11700
+Text Label -1400 4400 0    50   ~ 0
+G18
+Text Label -1400 4300 0    50   ~ 0
+G19
 Text Label -1400 4200 0    50   ~ 0
-G18
-Text Label -1400 4100 0    50   ~ 0
-G19
-Text Label -1400 4000 0    50   ~ 0
 G20
-NoConn ~ -1400 5600
-NoConn ~ -1400 5700
+NoConn ~ -1400 4000
+NoConn ~ -1400 4100
 NoConn ~ -1400 5800
 NoConn ~ -1400 5900
@@
 NoConn ~ -1400 11500
 $Comp
-L power:GND #PWR?
+L power:GND #PWR0149
 U 1 1 5D77F4DB
 P 1600 1100
-F 0 "#PWR?" H 1600 850 50  0001 C CNN
+F 0 "#PWR0149" H 1600 850 50  0001 C CNN
 F 1 "GND" H 1605 927 50  0000 C CNN
 F 2 "" H 1600 1100 50  0001 C CNN
@@
 $EndComp
 $Comp
-L power:GND #PWR?
+L power:GND #PWR0150
 U 1 1 5D77F5A3
 P 3500 1100
-F 0 "#PWR?" H 3500 850 50  0001 C CNN
+F 0 "#PWR0150" H 3500 850 50  0001 C CNN
 F 1 "GND" H 3505 927 50  0000 C CNN
 F 2 "" H 3500 1100 50  0001 C CNN
@@
 $EndComp
 $Comp
-L power:GND #PWR?
+L power:GND #PWR0151
 U 1 1 5D77FBAC
 P 7200 1100
-F 0 "#PWR?" H 7200 850 50  0001 C CNN
+F 0 "#PWR0151" H 7200 850 50  0001 C CNN
 F 1 "GND" H 7205 927 50  0000 C CNN
 F 2 "" H 7200 1100 50  0001 C CNN
@@
 $EndComp
 $Comp
-L power:GND #PWR?
+L power:GND #PWR0152
 U 1 1 5D77FDF3
 P 8300 1100
-F 0 "#PWR?" H 8300 850 50  0001 C CNN
+F 0 "#PWR0152" H 8300 850 50  0001 C CNN
 F 1 "GND" H 8305 927 50  0000 C CNN
 F 2 "" H 8300 1100 50  0001 C CNN
@@
 $EndComp
 $Comp
-L power:GND #PWR?
+L power:GND #PWR0153
 U 1 1 5D78018C
 P 10100 1100
-F 0 "#PWR?" H 10100 850 50  0001 C CNN
+F 0 "#PWR0153" H 10100 850 50  0001 C CNN
 F 1 "GND" H 10105 927 50  0000 C CNN
 F 2 "" H 10100 1100 50  0001 C CNN

Commit message: remove global labels
Connections:
- net labels added: SPI_Grids_Anodes
- net labels removed: SPI_Grids_Anodes_A
Changed lines of the file:
@@
 $EndComp
 Text HLabel -2250 1000 0    50   Input ~ 0
-SPI_Grids_Anodes_A
+SPI_Grids_Anodes
 Text HLabel -2400 600  0    50   Input ~ 0
 SRCLK
@@
 Text Label -2200 7100 2    50   ~ 0
 RCLK
-Text GLabel 1500 1100 0    50   Input ~ 0
-Filament_In_B
-Text GLabel 10200 1100 2    50   Input ~ 0
-Filament_In_A
 $Comp
 L power:GND #PWR056
@@
 	1    0    0    -1
 $EndComp
+Text HLabel 1500 1100 0    50   Input ~ 0
+Filament_In_B
+Text HLabel 10200 1100 2    50   Input ~ 0
+Filament_In_A
 $EndSCHEMATC
