File: vfd_stm32/vfd_stm32.kicad_pcb (KiCad board)
At the start: 2 copper layers, 1 part, among them U1 DC201LA

Commit message: cleanup electronics
Parts:
- added C1: 10u, Capacitor_SMD:C_1206_3216Metric_Pad1.42x1.75mm_HandSolder, F.Cu at (194.0, 41.4)
- added C10: 100n, Capacitor_SMD:C_0805_2012Metric_Pad1.15x1.40mm_HandSolder, F.Cu at (321.4, 50.2)
- added C11: 100n, Capacitor_SMD:C_0805_2012Metric_Pad1.15x1.40mm_HandSolder, F.Cu at (339.2, 50.2)
- added C2: 100n, Capacitor_SMD:C_0805_2012Metric_Pad1.15x1.40mm_HandSolder, F.Cu at (190.6, 40.8)
- added C3: 2.2u, Capacitor_SMD:C_0805_2012Metric_Pad1.15x1.40mm_HandSolder, F.Cu at (189.4, 37.0)
- added C4: 100n, Capacitor_SMD:C_0805_2012Metric_Pad1.15x1.40mm_HandSolder, F.Cu at (42.0, 50.2)
- added C5: 100n, Capacitor_SMD:C_0805_2012Metric_Pad1.15x1.40mm_HandSolder, F.Cu at (59.8, 50.2)
- added C6: 100n, Capacitor_SMD:C_0805_2012Metric_Pad1.15x1.40mm_HandSolder, F.Cu at (77.6, 50.2)
- added C7: 100n, Capacitor_SMD:C_0805_2012Metric_Pad1.15x1.40mm_HandSolder, F.Cu at (97.8, 50.2)
- added C8: 100n, Capacitor_SMD:C_0805_2012Metric_Pad1.15x1.40mm_HandSolder, F.Cu at (283.2, 50.2)
- added C9: 100n, Capacitor_SMD:C_0805_2012Metric_Pad1.15x1.40mm_HandSolder, F.Cu at (303.4, 50.2)
- added R1: 100k, Resistor_SMD:R_0805_2012Metric_Pad1.15x1.40mm_HandSolder, F.Cu at (180.8, 43.4)
- added R2: R_sense 500mW, Resistor_SMD:R_1206_3216Metric_Pad1.42x1.75mm_HandSolder, F.Cu at (178.0, 38.4)
- added U10: 74HC595, Package_SO:SOIC-16_3.9x9.9mm_P1.27mm, F.Cu at (289.6, 52.0)
- added U11: 74HC595, Package_SO:SOIC-16_3.9x9.9mm_P1.27mm, F.Cu at (309.8, 52.0)
- added U12: 74HC595, Package_SO:SOIC-16_3.9x9.9mm_P1.27mm, F.Cu at (327.8, 52.0)
- added U13: 74HC595, Package_SO:SOIC-16_3.9x9.9mm_P1.27mm, F.Cu at (345.6, 52.0)
- added U14: ULN2003, Package_SO:SOIC-16_3.9x9.9mm_P1.27mm, F.Cu at (288.2, 60.0)
- added U15: ULN2003, Package_SO:SOIC-16_3.9x9.9mm_P1.27mm, F.Cu at (308.6, 60.0)
- added U16: ULN2003, Package_SO:SOIC-16_3.9x9.9mm_P1.27mm, F.Cu at (326.4, 60.0)
- added U17: ULN2003, Package_SO:SOIC-16_3.9x9.9mm_P1.27mm, F.Cu at (344.2, 60.0)
- added U18: DRV8848, Package_SO:TSSOP-16-1EP_4.4x5mm_P0.65mm, F.Cu at (184.7, 39.3)
- added U19: STM32F303K8Tx, Package_QFP:LQFP-32_7x7mm_P0.8mm, F.Cu at (76.6, 34.4)
- added U2: 74HC595, Package_SO:SOIC-16_3.9x9.9mm_P1.27mm, F.Cu at (48.4, 52.0)
- added U3: 74HC595, Package_SO:SOIC-16_3.9x9.9mm_P1.27mm, F.Cu at (66.2, 52.0)
- added U4: 74HC595, Package_SO:SOIC-16_3.9x9.9mm_P1.27mm, F.Cu at (84.0, 52.0)
- added U5: 74HC595, Package_SO:SOIC-16_3.9x9.9mm_P1.27mm, F.Cu at (104.2, 52.0)
- added U6: ULN2003, Package_SO:SOIC-16_3.9x9.9mm_P1.27mm, F.Cu at (47.0, 60.0)
- added U7: ULN2003, Package_SO:SOIC-16_3.9x9.9mm_P1.27mm, F.Cu at (64.8, 60.0)
- added U8: ULN2003, Package_SO:SOIC-16_3.9x9.9mm_P1.27mm, F.Cu at (82.6, 60.0)
- added U9: ULN2003, Package_SO:SOIC-16_3.9x9.9mm_P1.27mm, F.Cu at (102.8, 60.0)
- moved U1 16.1 mm to (20.0, 20.0)
Connections:
- net /Filament_Voltage_A renamed /VFD/Filament_In_A
- net /Filament_Voltage_B renamed /VFD/Filament_In_B
Routing:
- net /VFD/Power_Grids_Anodes: track 0.00 -> 125.5 mm
- net GND: track 0.00 -> 125.5 mm
- net VCC: track 0.00 -> 16.1 mm
- net Net-(U1-Pad24): track 0.00 -> 8.42 mm
- net Net-(U1-Pad40): track 0.00 -> 8.35 mm
- net Net-(U1-Pad23): track 0.00 -> 7.15 mm
- net Net-(U1-Pad41): track 0.00 -> 7.08 mm
- net Net-(U1-Pad31): track 0.00 -> 5.94 mm
- net Net-(U1-Pad39): track 0.00 -> 5.93 mm
- net Net-(U1-Pad9): track 0.00 -> 5.92 mm
- net Net-(U1-Pad16): track 0.00 -> 5.90 mm
- net Net-(U1-Pad47): track 0.00 -> 5.90 mm
- net Net-(U1-Pad22): track 0.00 -> 5.89 mm
- net Net-(U1-Pad54): track 0.00 -> 5.89 mm
- net Net-(U1-Pad55): track 0.00 -> 5.88 mm
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- added copper zone on F.Cu, net GND

Commit message: routage terminé
Parts:
- removed the U12 at (327.8, 52.0)
- removed the U9 at (102.8, 60.0)
- added C12: 33n, Capacitor_SMD:C_0805_2012Metric_Pad1.15x1.40mm_HandSolder, F.Cu at (185.4, 33.8)
- added R3: 100, Resistor_SMD:R_0805_2012Metric_Pad1.15x1.40mm_HandSolder, F.Cu at (179.2, 36.4)
- added R4: 100, Resistor_SMD:R_0805_2012Metric_Pad1.15x1.40mm_HandSolder, F.Cu at (181.4, 36.4)
- added R5: 47k, Resistor_SMD:R_0805_2012Metric_Pad1.15x1.40mm_HandSolder, F.Cu at (177.2, 33.8)
- added R6: 47k, Resistor_SMD:R_0805_2012Metric_Pad1.15x1.40mm_HandSolder, F.Cu at (183.4, 33.8)
- added SW1: SW_DIP_x04, Button_Switch_SMD:SW_DIP_SPSTx04_Slide_6.7x11.72mm_W6.73mm_P2.54mm_LowProfile_JPin, F.Cu at (120.0, 32.4)
- added U13: 74HC595, Package_SO:SOIC-16_3.9x9.9mm_P1.27mm, F.Cu at (106.8, 51.4)
- added U16: 74HC595, Package_SO:SOIC-16_3.9x9.9mm_P1.27mm, F.Cu at (327.6, 51.4)
- added U20: STM32F302C8Tx, Package_QFP:LQFP-48_7x7mm_P0.5mm, F.Cu at (63.2, 32.6)
- C10, C11, C4, C5, C6, C7, C8, C9: moved to B.Cu
- U19: value STM32F303K8Tx -> TSZ121ILT; footprint Package_QFP:LQFP-32_7x7mm_P0.8mm -> Package_TO_SOT_SMD:SOT-23-5
- U5: value 74HC595 -> ULN2003
- moved U19 103.8 mm to (180.4, 32.4)
- moved C1 11.9 mm to (182.2, 43.2)
- moved C3 11.5 mm to (180.1, 43.8), turned to 270 degrees
- moved U18 11.0 mm to (182.0, 50.0), turned to 90 degrees
- moved C6 10.3 mm to (87.8, 51.4)
- moved C8 10.3 mm to (293.4, 51.4)
- moved R1 9.82 mm to (186.2, 51.6), turned to 90 degrees
- moved R2 9.42 mm to (177.4, 47.8), turned to 90 degrees
- moved C7 9.08 mm to (106.8, 51.4)
- moved C5 8.88 mm to (68.6, 51.4)
- moved U5 8.86 mm to (100.4, 60.0), turned to 270 degrees
- moved C11 7.69 mm to (346.8, 51.4)
- moved C4 7.69 mm to (49.6, 51.4)
- moved C2 6.80 mm to (184.5, 43.8)
- moved C10 6.34 mm to (327.6, 51.4)
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- renumbered U2 to U10, U3 to U11, U4 to U12, U10 to U14, U11 to U15, U13 to U17, U6 to U2, U7 to U3, U8 to U4, U14 to U6, U15 to U7, U16 to U8, U17 to U9
Connections:
- C1 pad 1: GNDPWR -> GND
- C10 pad 1: VCC -> +3V3
- C11 pad 1: VCC -> +3V3
- C2 pad 1: GNDPWR -> GND
- C3 pad 1: GNDPWR -> GND
- C4 pad 1: VCC -> +3V3
- C5 pad 1: VCC -> +3V3
- C6 pad 1: VCC -> +3V3
- C7 pad 1: VCC -> +3V3
- C8 pad 1: VCC -> +3V3
- C9 pad 1: VCC -> +3V3
- R2 pad 2: GNDPWR -> GND
- U1 pad 1: /VFD/Filament_In_B -> Filament_In_B
- U1 pad 2: Net-(U1-Pad2) -> GND
- U1 pad 21: Net-(U1-Pad21) -> GND
- U1 pad 32: Net-(U1-Pad32) -> GND
- U1 pad 43: Net-(U1-Pad43) -> GND
- U1 pad 61: Net-(U1-Pad61) -> GND
- U1 pad 62: /VFD/Filament_In_A -> Filament_In_A
- U10 pad 1: Net-(U2-Pad1) -> /VFD/P2
- U10 pad 10: VCC -> +3V3
- U10 pad 15: Net-(U2-Pad15) -> /VFD/P1
- U10 pad 16: VCC -> +3V3
- U10 pad 2: Net-(U2-Pad2) -> /VFD/P3
- U10 pad 3: Net-(U2-Pad3) -> /VFD/P4
- U10 pad 4: Net-(U2-Pad4) -> /VFD/P5
- U10 pad 5: Net-(U2-Pad5) -> /VFD/P6
- U10 pad 6: Net-(U2-Pad6) -> /VFD/P7
- U10 pad 7: Net-(U2-Pad7) -> /VFD/P8
- U11 pad 1: Net-(U3-Pad1) -> /VFD/P10
- U11 pad 10: VCC -> +3V3
- U11 pad 15: Net-(U3-Pad15) -> /VFD/P9
- U11 pad 16: VCC -> +3V3
- U11 pad 2: Net-(U3-Pad2) -> /VFD/P11
- U11 pad 3: Net-(U3-Pad3) -> /VFD/P12
- U11 pad 4: Net-(U3-Pad4) -> /VFD/P13
- U11 pad 5: Net-(U3-Pad5) -> /VFD/P14
- U11 pad 6: Net-(U3-Pad6) -> /VFD/P15
- U11 pad 7: Net-(U3-Pad7) -> /VFD/P16
- U12 pad 1: Net-(U4-Pad1) -> /VFD/P18
- U12 pad 10: VCC -> +3V3
- U12 pad 15: Net-(U4-Pad15) -> /VFD/P17
- U12 pad 16: VCC -> +3V3
- U12 pad 2: Net-(U4-Pad2) -> /VFD/G20
- U12 pad 3: Net-(U4-Pad3) -> /VFD/G19
- U12 pad 4: Net-(U4-Pad4) -> /VFD/G18
- U12 pad 5: Net-(U4-Pad5) -> /VFD/G17
- U12 pad 6: Net-(U4-Pad6) -> /VFD/G16
- U12 pad 7: Net-(U4-Pad7) -> /VFD/G15
- U12 pad 9: Net-(U4-Pad9) -> Net-(U12-Pad9)
- U14 pad 1: Net-(U10-Pad1) -> /VFD/G9
- U14 pad 10: VCC -> +3V3
- U14 pad 14: /VFD/SPI_Grids_Anodes_B -> Net-(U13-Pad9)
- U14 pad 15: Net-(U10-Pad15) -> /VFD/G10
- U14 pad 16: VCC -> +3V3
- U14 pad 2: Net-(U10-Pad2) -> /VFD/G8
- U14 pad 3: Net-(U10-Pad3) -> /VFD/G7
- U14 pad 4: Net-(U10-Pad4) -> /VFD/G6
- U14 pad 5: Net-(U10-Pad5) -> /VFD/G5
- U14 pad 6: Net-(U10-Pad6) -> /VFD/G4
- U14 pad 7: Net-(U10-Pad7) -> /VFD/G3
- U15 pad 1: Net-(U11-Pad1) -> /VFD/G1
- U15 pad 10: VCC -> +3V3
- U15 pad 15: Net-(U11-Pad15) -> /VFD/G2
- U15 pad 16: VCC -> +3V3
- U15 pad 2: Net-(U11-Pad2) -> Net-(U15-Pad2)
- U15 pad 3: Net-(U11-Pad3) -> Net-(U15-Pad3)
- U15 pad 4: Net-(U11-Pad4) -> Net-(U15-Pad4)
- U15 pad 5: Net-(U11-Pad5) -> /VFD/P35
- U15 pad 6: Net-(U11-Pad6) -> /VFD/P34
- U15 pad 7: Net-(U11-Pad7) -> /VFD/P33
- U17 pad 1: Net-(U13-Pad1) -> /VFD/P23
- U17 pad 10: VCC -> +3V3
- U17 pad 15: Net-(U13-Pad15) -> /VFD/P24
- U17 pad 16: VCC -> +3V3
- U17 pad 2: Net-(U13-Pad2) -> /VFD/P22
- U17 pad 3: Net-(U13-Pad3) -> /VFD/P21
- U17 pad 4: Net-(U13-Pad4) -> /VFD/P20
- U17 pad 5: Net-(U13-Pad5) -> /VFD/P19
- U17 pad 6: Net-(U13-Pad6) -> Net-(U17-Pad6)
- U17 pad 7: Net-(U13-Pad7) -> Net-(U17-Pad7)
- U18 pad 13: GNDPWR -> GND
- U18 pad 17: GNDPWR -> GND
- U18 pad 2: /Filament_In_A -> Filament_In_A
- U18 pad 4: /Filament_In_B -> Filament_In_B
- U18 pad 5: /Filament_In_B -> Filament_In_B
- U18 pad 7: /Filament_In_A -> Filament_In_A
- U19 pad 1: VDD -> /Filament_ADC
- U19 pad 2: Net-(U19-Pad2) -> GND
- U19 pad 5: Net-(U19-Pad5) -> +3V3
- U2 pad 1: Net-(U2-Pad7) -> /VFD/P7
- U2 pad 2: Net-(U2-Pad6) -> /VFD/P6
- U2 pad 3: Net-(U2-Pad5) -> /VFD/P5
- U2 pad 4: Net-(U2-Pad4) -> /VFD/P4
- U2 pad 5: Net-(U2-Pad3) -> /VFD/P3
- U2 pad 6: Net-(U2-Pad2) -> /VFD/P2
- U2 pad 7: Net-(U2-Pad1) -> /VFD/P1
- U3 pad 1: Net-(U3-Pad7) -> /VFD/P14
- U3 pad 2: Net-(U3-Pad6) -> /VFD/P13
- U3 pad 3: Net-(U3-Pad5) -> /VFD/P12
- U3 pad 4: Net-(U3-Pad4) -> /VFD/P11
- U3 pad 5: Net-(U3-Pad3) -> /VFD/P10
- U3 pad 6: Net-(U3-Pad2) -> /VFD/P9
- U3 pad 7: Net-(U3-Pad1) -> /VFD/P8
- U4 pad 1: Net-(U4-Pad7) -> /VFD/G18
- U4 pad 2: Net-(U4-Pad6) -> /VFD/G19
- U4 pad 3: Net-(U4-Pad5) -> /VFD/G20
- U4 pad 4: Net-(U4-Pad4) -> /VFD/P18
- U4 pad 5: Net-(U4-Pad3) -> /VFD/P17
- U4 pad 6: Net-(U4-Pad2) -> /VFD/P16
- U4 pad 7: Net-(U4-Pad1) -> /VFD/P15
- U5 pad 1: Net-(U5-Pad1) -> /VFD/G11
- U5 pad 10: VCC -> Net-(U1-Pad25)
- U5 pad 11: /VFD/SRCLK -> Net-(U1-Pad26)
- U5 pad 12: /VFD/RCLK -> Net-(U1-Pad27)
- U5 pad 13: GND -> Net-(U1-Pad28)
- U5 pad 14: Net-(U4-Pad9) -> Net-(U1-Pad29)
- U5 pad 15: Net-(U5-Pad15) -> Net-(U1-Pad30)
- U5 pad 16: VCC -> Net-(U1-Pad31)
- U5 pad 2: Net-(U5-Pad2) -> /VFD/G12
- U5 pad 3: Net-(U5-Pad3) -> /VFD/G13
- U5 pad 4: Net-(U5-Pad4) -> /VFD/G14
- U5 pad 5: Net-(U5-Pad5) -> /VFD/G15
- U5 pad 6: Net-(U5-Pad6) -> /VFD/G16
- U5 pad 7: Net-(U5-Pad7) -> /VFD/G17
- U5 pad 9: /VFD/SPI_Grids_Anodes_B -> /VFD/Power_Grids_Anodes
- U6 pad 1: Net-(U10-Pad7) -> /VFD/G4
- U6 pad 2: Net-(U10-Pad6) -> /VFD/G5
- U6 pad 3: Net-(U10-Pad5) -> /VFD/G6
- U6 pad 4: Net-(U10-Pad4) -> /VFD/G7
- U6 pad 5: Net-(U10-Pad3) -> /VFD/G8
- U6 pad 6: Net-(U10-Pad2) -> /VFD/G9
- U6 pad 7: Net-(U10-Pad1) -> /VFD/G10
- U7 pad 1: Net-(U11-Pad7) -> /VFD/P32
- U7 pad 2: Net-(U11-Pad6) -> /VFD/P33
- U7 pad 3: Net-(U11-Pad5) -> /VFD/P34
- U7 pad 4: Net-(U11-Pad4) -> /VFD/P35
- U7 pad 5: Net-(U11-Pad3) -> /VFD/G1
- U7 pad 6: Net-(U11-Pad2) -> /VFD/G2
- U7 pad 7: Net-(U11-Pad1) -> /VFD/G3
- U8 pad 1: Net-(U12-Pad7) -> /VFD/P25
- U8 pad 2: Net-(U12-Pad6) -> /VFD/P26
- U8 pad 3: Net-(U12-Pad5) -> /VFD/P27
- U8 pad 4: Net-(U12-Pad4) -> /VFD/P28
- U8 pad 5: Net-(U12-Pad3) -> /VFD/P29
- U8 pad 6: Net-(U12-Pad2) -> /VFD/P30
- U8 pad 7: Net-(U12-Pad1) -> /VFD/P31
- U9 pad 1: Net-(U13-Pad7) -> Net-(U9-Pad1)
- U9 pad 2: Net-(U13-Pad6) -> /VFD/P19
- U9 pad 3: Net-(U13-Pad5) -> /VFD/P20
- U9 pad 4: Net-(U13-Pad4) -> /VFD/P21
- U9 pad 5: Net-(U13-Pad3) -> /VFD/P22
- U9 pad 6: Net-(U13-Pad2) -> /VFD/P23
- U9 pad 7: Net-(U13-Pad1) -> /VFD/P24
Routing:
- net /VFD/RCLK: track 0.00 -> 324.5 mm, vias 0 -> 14
- net /VFD/SRCLK: track 0.00 -> 320.5 mm
- net GND: track 125.5 -> 345.3 mm, vias 0 -> 9
- net Filament_In_A: track 0.00 -> 206.8 mm, vias 0 -> 4
- net Net-(U13-Pad9): track 0.00 -> 189.0 mm
- net /VFD/Power_Grids_Anodes: track 125.5 -> 310.1 mm
- net Filament_In_B: track 0.00 -> 178.5 mm
- net +3V3: track 0.00 -> 172.7 mm, vias 0 -> 17
- net /VFD/SPI_Grids_Anodes_A: track 0.00 -> 65.5 mm
- net Net-(R2-Pad1): track 0.00 -> 30.8 mm, vias 0 -> 2
- net /VFD/P32: track 0.00 -> 17.0 mm
- net VCC: track 16.1 -> 0.00 mm
- net Net-(U16-Pad9): track 0.00 -> 14.0 mm
- net Net-(U11-Pad9): track 0.00 -> 14.0 mm
- net Net-(U15-Pad9): track 0.00 -> 13.8 mm
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- added copper zone on B.Cu, net GND
Other:
- board outline added: 346 x 48 mm

Commit message: Fix shift registers outputs. Add text description files
Parts:
- moved C6 2.60 mm to (85.2, 51.4)
- moved C7 2.60 mm to (104.2, 51.4)
- moved U12 2.60 mm to (85.2, 51.4)
- moved U13 2.60 mm to (104.2, 51.4)
Connections:
- U12 pad 2: /VFD/G20 -> Net-(U12-Pad2)
- U12 pad 3: /VFD/G19 -> Net-(U12-Pad3)
- U12 pad 4: /VFD/G18 -> /VFD/G20
- U12 pad 5: /VFD/G17 -> /VFD/G19
- U12 pad 6: /VFD/G16 -> /VFD/G18
- U12 pad 7: /VFD/G15 -> /VFD/G17
- U13 pad 1: /VFD/G13 -> /VFD/G15
- U13 pad 15: /VFD/G14 -> /VFD/G16
- U13 pad 2: /VFD/G12 -> /VFD/G14
- U13 pad 3: /VFD/G11 -> /VFD/G13
- U13 pad 4: Net-(U13-Pad4) -> /VFD/G12
- U13 pad 5: Net-(U13-Pad5) -> /VFD/G11
Routing:
- net /VFD/G15: track 11.0 -> 3.20 mm
- net /VFD/G14: track 9.67 -> 3.20 mm
- net Net-(U13-Pad9): track 189.0 -> 191.6 mm
- net Net-(U11-Pad9): track 14.0 -> 11.4 mm
- net /VFD/SRCLK: track 320.5 -> 322.8 mm
- net /VFD/G16: track 11.3 -> 9.65 mm
- net /VFD/P18: track 3.25 -> 4.23 mm
- net /VFD/P17: track 9.70 -> 10.3 mm

Commit message: reroute a bit
Parts:
- moved U20 88.2 mm to (138.0, -14.2)
- moved SW1 58.9 mm to (157.6, -13.0)
- moved C1 8.09 mm to (187.4, 37.0)
- moved R1 8.09 mm to (191.4, 45.4)
- moved R3 8.09 mm to (184.4, 30.2)
- moved C3 8.09 mm to (185.3, 37.6)
- moved R5 8.09 mm to (182.4, 27.6)
- moved U18 8.09 mm to (187.2, 43.8)
- moved R4 8.09 mm to (186.6, 30.2)
- moved U19 8.09 mm to (185.6, 26.2)
- moved C12 8.09 mm to (190.6, 27.6)
- moved C2 8.09 mm to (189.7, 37.6)
- moved R2 8.09 mm to (182.6, 41.6)
- moved R6 8.09 mm to (188.6, 27.6)
Routing:
- net +3V3: track 172.7 -> 343.3 mm, vias 17 -> 19
- net Filament_In_A: track 206.8 -> 199.7 mm
- net Filament_In_B: track 178.5 -> 181.1 mm
Other:
- board size 346 x 48 mm -> 326 x 48 mm
