File: vfd_stm32/vfd_display.kicad_pcb (KiCad board)
At the start: 2 copper layers, 326 x 48 mm, 39 parts, among them SW1 SW_DIP_x04, U1 DC201LA, U10 74HC595, U11 74HC595, U12 74HC595, U13 74HC595, U14 74HC595, U15 74HC595, U16 74HC595, U17 74HC595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

Commit message: continue circuitry
Parts:
- added C13: 100n, Capacitor_SMD:C_0805_2012Metric_Pad1.15x1.40mm_HandSolder, F.Cu at (54.6, 60.0)
- added C14: 100n, Capacitor_SMD:C_0805_2012Metric_Pad1.15x1.40mm_HandSolder, F.Cu at (72.4, 60.0)
- added C15: 100n, Capacitor_SMD:C_0805_2012Metric_Pad1.15x1.40mm_HandSolder, F.Cu at (90.2, 60.0)
- added C16: 100n, Capacitor_SMD:C_0805_2012Metric_Pad1.15x1.40mm_HandSolder, F.Cu at (108.0, 60.0)
- added C17: 100n, Capacitor_SMD:C_0805_2012Metric_Pad1.15x1.40mm_HandSolder, F.Cu at (283.2, 60.0)
- added C18: 100n, Capacitor_SMD:C_0805_2012Metric_Pad1.15x1.40mm_HandSolder, F.Cu at (301.0, 60.0)
- added C19: 100n, Capacitor_SMD:C_0805_2012Metric_Pad1.15x1.40mm_HandSolder, F.Cu at (318.8, 60.0)
- added C20: 100n, Capacitor_SMD:C_0805_2012Metric_Pad1.15x1.40mm_HandSolder, F.Cu at (336.6, 60.0)
- R1: value 100k -> 10k
- moved R5 24.8 mm to (186.3, 52.1), turned to 0 degrees
- moved U19 22.7 mm to (184.9, 48.9), turned to 90 degrees
- moved R3 20.4 mm to (188.9, 50.1), turned to 0 degrees
- moved R6 18.4 mm to (186.3, 45.9), turned to 0 degrees
- moved R4 17.8 mm to (188.9, 47.9), turned to 0 degrees
- moved C12 16.8 mm to (186.3, 43.9), turned to 0 degrees
- moved C1 13.7 mm to (199.6, 43.2), turned to 180 degrees
- moved R2 13.0 mm to (193.4, 48.8)
- moved R1 12.9 mm to (203.0, 51.0), turned to 0 degrees
- moved U18 11.7 mm to (197.8, 48.8)
- moved C3 11.3 mm to (195.0, 43.4), turned to 0 degrees
- moved C2 10.0 mm to (199.2, 40.8), turned to 180 degrees
Connections:
- net /VFD/Power_Grids_Anodes renamed /Grids_Anodes_Power
- net /VFD/RCLK renamed /Logic/Grids_Anodes_SPI_RCLK
- net /VFD/SPI_Grids_Anodes_A renamed /Logic/Grids_Anodes_SPI_MOSI
- net /VFD/SRCLK renamed /Logic/Grids_Anodes_SPI_SRCLK
- net Filament_In_A renamed /VFD/Filament_In_A
- net Filament_In_B renamed /VFD/Filament_In_B
- net Net-(U18-Pad1) renamed /Logic/Filament_Enable
- net Net-(U18-Pad10) renamed /Logic/Filament_PWM2
- net Net-(U18-Pad9) renamed /Logic/Filament_PWM1
Routing:
- net /VFD/Filament_In_B: track 181.1 -> 251.1 mm
- net Net-(R2-Pad1): track 30.8 -> 10.9 mm, vias 2 -> 0
- net /VFD/Filament_In_A: track 199.7 -> 188.7 mm, vias 4 -> 2
- net GND: track 345.3 -> 337.3 mm
- net +3V3: track 343.3 -> 338.9 mm, vias 19 -> 18

Commit message: todo
Connections:
- U10 pad 11: /Logic/Grids_Anodes_SPI_SRCLK -> /VFD/SRCLK1
- U10 pad 12: /Logic/Grids_Anodes_SPI_RCLK -> /VFD/RCLK1
- U11 pad 11: /Logic/Grids_Anodes_SPI_SRCLK -> /VFD/SRCLK1
- U11 pad 12: /Logic/Grids_Anodes_SPI_RCLK -> /VFD/RCLK1
- U12 pad 11: /Logic/Grids_Anodes_SPI_SRCLK -> /VFD/SRCLK1
- U12 pad 12: /Logic/Grids_Anodes_SPI_RCLK -> /VFD/RCLK1
- U13 pad 11: /Logic/Grids_Anodes_SPI_SRCLK -> /VFD/SRCLK1
- U13 pad 12: /Logic/Grids_Anodes_SPI_RCLK -> /VFD/RCLK1
- U13 pad 9: Net-(U13-Pad9) -> /VFD/SPI_Grids_Anodes_1_out
- U14 pad 11: /Logic/Grids_Anodes_SPI_SRCLK -> /VFD/SRCLK2
- U14 pad 12: /Logic/Grids_Anodes_SPI_RCLK -> /VFD/RCLK2
- U14 pad 14: Net-(U13-Pad9) -> /VFD/SPI_Grids_Anodes_2
- U15 pad 11: /Logic/Grids_Anodes_SPI_SRCLK -> /VFD/SRCLK2
- U15 pad 12: /Logic/Grids_Anodes_SPI_RCLK -> /VFD/RCLK2
- U16 pad 11: /Logic/Grids_Anodes_SPI_SRCLK -> /VFD/SRCLK2
- U16 pad 12: /Logic/Grids_Anodes_SPI_RCLK -> /VFD/RCLK2
- U17 pad 11: /Logic/Grids_Anodes_SPI_SRCLK -> /VFD/SRCLK2
- U17 pad 12: /Logic/Grids_Anodes_SPI_RCLK -> /VFD/RCLK2
Routing:
- net /Logic/Grids_Anodes_SPI_RCLK: track 324.5 -> 0.00 mm, vias 14 -> 0
- net /Logic/Grids_Anodes_SPI_SRCLK: track 322.8 -> 0.00 mm
- net Net-(U13-Pad9): track 191.6 -> 0.00 mm
- net +3V3: track 338.9 -> 170.7 mm
- net /VFD/RCLK2: track 0.00 -> 71.6 mm, vias 0 -> 8
- net /VFD/SRCLK1: track 0.00 -> 70.3 mm
- net /VFD/SRCLK2: track 0.00 -> 70.1 mm
- net /VFD/RCLK1: track 0.00 -> 70.1 mm, vias 0 -> 6
- net /VFD/SPI_Grids_Anodes_2: track 0.00 -> 6.61 mm
- net /VFD/SPI_Grids_Anodes_1_out: track 0.00 -> 3.86 mm
