File: vfd_stm32/vfd_display.sch (KiCad schematic (older format))
At the start: 12 parts, among them U18 DRV8848, U19 TSZ121ILT

Commit message: continue circuitry
Parts:
- R1: value 100k -> 10k
Connections:
- net labels added: +5V, Grids_Anodes_Power
- net labels removed: Filament_In_A, Filament_In_B
- wire segments 32 -> 53
- no-connect marks 2 -> 3
Other:
- moved on the sheet: C1, C12, C2, C3, R1, R2, R3, R4, R5, R6, U18
