File: vfd_display.kicad_pcb (KiCad board)
At the start: 2 copper layers, 326 x 48 mm, 47 parts, among them SW1 SW_DIP_x04, U1 DC201LA, U10 74HC595, U11 74HC595, U12 74HC595, U13 74HC595, U14 74HC595, U15 74HC595, U16 74HC595, U17 74HC595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

Commit message: Bump to Kicad 6!
Other:
- net class Default removed
